File: abx.kicad_pcb (KiCad board)
At the start: 2 copper layers, 100 x 100 mm, 73 parts, among them CON1 PJ-307, CON2 PJ-307, CON3 PJ-307, CON4 2.1x5.5mm, IC1 ARDUINO_NANO, K1 FTR-B3GB003Z, K2 FTR-B3GB003Z, K3 FTR-B3GB003Z, K4 FTR-B3GB003Z, K5 FTR-B3GB003Z, K6 FTR-B3GB003Z, P1 CONN_2X1, Q1 BS250, Q10 2N7000, Q11 BS250, Q12 2N7000, Q2 2N7000, Q3 BS250, Q4 2N7000, Q5 BS250, Q6 2N7000, Q7 BS250, Q8 2N7000, Q9 BS250, SW1 SWITCH, SW2 REVEAL, SW3 REROLL

Commit message: board revision 3
Parts:
- removed CON1, CON2: PJ-307, SJ1-3523N
- added IN_X1: PJ-307, SJ1-3523N, F.Cu at (88.0, 150.0)
- added IN_Y1: PJ-307, SJ1-3523N, F.Cu at (103.0, 150.0)
- added P2: YL, 1pin_032_058, F.Cu at (112.4, 158.8)
- added P3: YR, 1pin_032_058, F.Cu at (117.5, 158.8)
- added P4: YG, 1pin_032_058, F.Cu at (114.9, 151.1)
- added P5: XL, 1pin_032_058, F.Cu at (78.7, 168.3)
- added P6: XR, 1pin_032_058, F.Cu at (86.4, 168.3)
- added P7: XG, 1pin_032_058, F.Cu at (78.7, 160.7)
Connections:
- IC1 pad 1: (no net) -> PCH4
- IC1 pad 2: (no net) -> NCH3
- IC1 pad 25: NCH3 -> (no net)
- IC1 pad 26: PCH4 -> (no net)
Routing:
- net N-0000050: track 43.0 -> 58.9 mm
- net N-0000048: track 52.4 -> 65.4 mm
- net N-0000025: track 53.0 -> 65.9 mm
- net N-0000047: track 61.1 -> 73.6 mm
- net N-0000041: track 58.7 -> 70.2 mm
- net N-0000026: track 59.2 -> 69.7 mm
- net 9V: track 275.1 -> 269.9 mm
- net NCH3: track 33.4 -> 38.3 mm
- net PCH4: track 45.3 -> 49.5 mm, vias 0 -> 2
Other:
- board text added: "Pepas Labs ABX-tayda v3"
- board text added: "XG"
- board text added: "XL"
- board text added: "XR"
- board text added: "YG"
- board text added: "YL"
- board text added: "YR"
- board text removed: "Pepas Labs ABX-tayda v2"

Commit message: v4
Parts:
- added R23: 10k, R_AXIAL_0W25_059A_PL, F.Cu at (155.6, 175.3)
- added R24: 10k, R_AXIAL_0W25_059A_PL, F.Cu at (154.9, 169.5)
- added R25: 10k, R_AXIAL_0W25_059A_PL, F.Cu at (158.1, 188.0)
- added R26: 10k, R_AXIAL_0W25_059A_PL, F.Cu at (160.7, 198.1)
- added R27: 10k, R_AXIAL_0W25_059A_PL, F.Cu at (155.6, 188.0)
- Q1, Q11, Q3, Q5, Q7, Q9: value BS250 -> 2N3906; footprint TO-92_Q_SGD_059Bo_PL -> TO-92_Q_EBC_059Bo_PL
Connections:
- IC1 pad 12: PCH2 -> N-0000025
- IC1 pad 14: PCH5 -> N-0000031
- IC1 pad 20: PCH6 -> N-0000040
- IC1 pad 22: PCH1 -> N-0000047
- IC1 pad 24: PCH3 -> N-0000046
Routing:
- net PCH6: track 32.5 -> 56.6 mm, vias 0 -> 1
- net PCH5: track 81.7 -> 64.4 mm
- net PCH2: track 51.1 -> 34.3 mm
- net N-0000031: track 0.00 -> 13.1 mm
- net N-0000046: track 0.00 -> 12.9 mm
- net N-0000025: track 0.00 -> 12.1 mm
- net PCH1: track 65.5 -> 76.3 mm
- net N-0000047: track 0.00 -> 10.4 mm
- net PCH3: track 35.3 -> 40.1 mm
- net N-0000038: track 28.9 -> 33.6 mm
- net N-0000040: track 0.00 -> 3.17 mm
- net N-000008: track 47.1 -> 49.9 mm
- net N-0000037: track 58.9 -> 59.9 mm
- net N-0000043: track 73.6 -> 72.7 mm
Other:
- board text added: "Pepas Labs ABX-tayda v4"
- board text removed: "Pepas Labs ABX-tayda v3"

Commit message: 4.1
Parts:
- added R28: 10k, R_AXIAL_0W25_059A_PL, F.Cu at (155.6, 219.1)
Connections:
- net PCH1 renamed PNP1
- net PCH2 renamed PNP2
- net PCH3 renamed PNP3
- net PCH5 renamed PNP5
- net PCH6 renamed PNP6
- IC1 pad 1: PCH4 -> N-0000034
- Q7 pad 2: PCH4 -> PNP4
- R14 pad 2: PCH4 -> PNP4
Routing:
- net PCH4: track 49.5 -> 0.00 mm, vias 2 -> 0
- net PNP4: track 0.00 -> 35.6 mm, vias 0 -> 1
- net N-0000034: track 0.00 -> 6.50 mm
Other:
- board text added: "Pepas Labs ABX-tayda v4.1"
- board text removed: "Pepas Labs ABX-tayda v4"
